File: eagle/badge.brd (EAGLE design)
At the start: 57.1 x 80 mm, 9 parts, among them IC1 TINY13-20PU

Commit message: updated schematic/board with correct VDD wiring
Might not be in sync now (between schematic and board), but the data is
correct. The problem was the battery output and switch output
accidentally had the same label, so the switch was being bypassed.
Correct this routing, as well as routing VDD to \bar{RESET} so we
wouldn't have to lose that functionality by changing RESET to a GPIO
Connections:
- net VDD: now also IC1.1
Routing:
- net VDD: track 95.2 -> 119.4 mm
Changed lines of the file:
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@@
 <contactref element="IC1" pad="8"/>
 <wire x1="16.53" y1="10.16" x2="16.51" y2="10.16" width="0.6096" layer="1"/>
-<wire x1="16.51" y1="17.78" x2="16.51" y2="33.02" width="0.6096" layer="1"/>
-<wire x1="16.51" y1="33.02" x2="29.21" y2="33.02" width="0.6096" layer="1"/>
-<wire x1="29.21" y1="33.02" x2="29.21" y2="30.48" width="0.6096" layer="1"/>
 <wire x1="24.17" y1="49.53" x2="26.67" y2="49.53" width="0.6096" layer="1"/>
-<wire x1="26.67" y1="49.53" x2="26.67" y2="43.18" width="0.6096" layer="1"/>
-<wire x1="26.67" y1="43.18" x2="29.21" y2="43.18" width="0.6096" layer="1"/>
-<wire x1="29.21" y1="43.18" x2="31.75" y2="43.18" width="0.6096" layer="1"/>
-<wire x1="31.75" y1="43.18" x2="31.75" y2="33.02" width="0.6096" layer="1"/>
-<wire x1="31.75" y1="33.02" x2="29.21" y2="33.02" width="0.6096" layer="1"/>
 <wire x1="39.37" y1="10.16" x2="39.37" y2="17.78" width="0.6096" layer="1"/>
 <via x="39.37" y="17.78" extent="1-16" drill="0.6" shape="square"/>
@@
 <via x="16.51" y="17.78" extent="1-16" drill="0.6" shape="square"/>
 <wire x1="16.51" y1="10.16" x2="16.51" y2="17.78" width="0.6096" layer="1"/>
+<wire x1="26.67" y1="49.53" x2="29.21" y2="43.18" width="0" layer="19" extent="1-1"/>
+<wire x1="29.21" y1="30.48" x2="29.21" y2="43.18" width="0" layer="19" extent="1-1"/>
+<wire x1="39.37" y1="17.78" x2="29.21" y2="30.48" width="0" layer="19" extent="1-1"/>
+<wire x1="16.51" y1="17.78" x2="16.51" y2="46.99" width="0.6096" layer="1"/>
+<wire x1="16.51" y1="46.99" x2="26.67" y2="46.99" width="0.6096" layer="1"/>
+<wire x1="26.67" y1="46.99" x2="26.67" y2="49.53" width="0.6096" layer="1"/>
+<wire x1="24.13" y1="49.53" x2="24.13" y2="45.72" width="0.6096" layer="16"/>
+<wire x1="24.13" y1="45.72" x2="29.21" y2="45.72" width="0.6096" layer="16"/>
+<wire x1="29.21" y1="45.72" x2="29.21" y2="43.18" width="0.6096" layer="16"/>
+<wire x1="29.21" y1="43.18" x2="26.67" y2="43.18" width="0.6096" layer="16"/>
+<wire x1="26.67" y1="43.18" x2="26.67" y2="30.48" width="0.6096" layer="16"/>
+<wire x1="26.67" y1="30.48" x2="29.21" y2="30.48" width="0.6096" layer="16"/>
+<contactref element="IC1" pad="1"/>
+<wire x1="29.21" y1="30.48" x2="21.59" y2="30.48" width="0.6096" layer="1"/>
 </signal>
 <signal name="GND">
