File: eagle/badge.sch (EAGLE design)
At the start: 9 parts, among them IC1 TINY13-20PU

Commit message: updated schematic/board with correct VDD wiring
Might not be in sync now (between schematic and board), but the data is
correct. The problem was the battery output and switch output
accidentally had the same label, so the switch was being bypassed.
Correct this routing, as well as routing VDD to \bar{RESET} so we
wouldn't have to lose that functionality by changing RESET to a GPIO
Connections:
- new net BATTERY: U$1.VDD_1, U$1.VDD_2, U$2.COMM
- net VDD: now also IC1.PB5/PCINT5/!RESET!/ADC0/DW; no longer U$1.VDD_1, U$1.VDD_2, U$2.COMM
Changed lines of the file:
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@@
 <net name="VDD" class="0">
-<segment>
-<pinref part="U$1" gate="G$1" pin="VDD_1"/>
-<wire x1="-33.02" y1="71.12" x2="-27.94" y2="71.12" width="0.1524" layer="91"/>
-<pinref part="U$1" gate="G$1" pin="VDD_2"/>
-<wire x1="-33.02" y1="68.58" x2="-27.94" y2="68.58" width="0.1524" layer="91"/>
-<wire x1="-27.94" y1="68.58" x2="-27.94" y2="71.12" width="0.1524" layer="91"/>
-<pinref part="U$2" gate="G$1" pin="COMM"/>
-<wire x1="-27.94" y1="71.12" x2="-20.32" y2="71.12" width="0.1524" layer="91"/>
-<junction x="-27.94" y="71.12"/>
-</segment>
 <segment>
 <pinref part="PHOTO_CELL" gate="G$1" pin="2"/>
@@
 <wire x1="25.4" y1="71.12" x2="27.94" y2="71.12" width="0.1524" layer="91"/>
 <label x="17.78" y="76.2" size="1.778" layer="95"/>
+</segment>
+<segment>
+<pinref part="IC1" gate="G$1" pin="PB5/PCINT5/!RESET!/ADC0/DW"/>
+<wire x1="27.94" y1="55.88" x2="17.78" y2="55.88" width="0.1524" layer="91"/>
+<label x="17.78" y="55.88" size="1.778" layer="95"/>
 </segment>
 </net>
@@
 </segment>
 </net>
+<net name="BATTERY" class="0">
+<segment>
+<pinref part="U$1" gate="G$1" pin="VDD_1"/>
+<wire x1="-33.02" y1="71.12" x2="-27.94" y2="71.12" width="0.1524" layer="91"/>
+<pinref part="U$1" gate="G$1" pin="VDD_2"/>
+<wire x1="-33.02" y1="68.58" x2="-27.94" y2="68.58" width="0.1524" layer="91"/>
+<wire x1="-27.94" y1="68.58" x2="-27.94" y2="71.12" width="0.1524" layer="91"/>
+<pinref part="U$2" gate="G$1" pin="COMM"/>
+<wire x1="-27.94" y1="71.12" x2="-20.32" y2="71.12" width="0.1524" layer="91"/>
+<junction x="-27.94" y="71.12"/>
+<label x="-27.94" y="76.2" size="1.778" layer="95"/>
+</segment>
+</net>
